Commit message: Initial urdf changes

File: turtlebot4_description/urdf/lite/turtlebot4.urdf.xacro (robot description, xacro)
@@ -24,6 +24,9 @@
     <origin xyz="${camera_mount_x_offset} ${camera_mount_y_offset} ${camera_mount_z_offset + base_link_z_offset}"/>
   </xacro:camera_bracket>
-  <xacro:oakd_lite name="oakd_lite" parent_link="oakd_lite_camera_bracket">
-    <origin xyz="${oakd_lite_x_offset} ${oakd_lite_y_offset} ${oakd_lite_z_offset}"/>
+  <xacro:oakd_lite name="oakd_lite" parent_link="oakd_lite_camera_bracket"
+                   cam_pos_x="${oakd_lite_x_offset}"
+                   cam_pos_y="${oakd_lite_y_offset}"
+                   cam_pos_z="${oakd_lite_z_offset}"
+                   cam_roll="0.0" cam_pitch="0.0" cam_yaw="0.0">
   </xacro:oakd_lite>
 </robot>

File: turtlebot4_description/urdf/sensors/oakd_lite.urdf.xacro (robot description, xacro)
@@ -1,6 +1,7 @@
 <?xml version="1.0"?>
 <robot xmlns:xacro="http://ros.org/wiki/xacro">
-<xacro:macro name="oakd_lite" params="name parent_link *origin">
+<xacro:macro name="oakd_lite" params="name parent_link cam_pos_x cam_pos_y cam_pos_z cam_roll cam_pitch cam_yaw">
   <xacro:include filename="$(find irobot_create_description)/urdf/common_properties.urdf.xacro"/>
+  <xacro:include filename="$(find depthai_bridge)/urdf/include/depthai_macro.urdf.xacro"/>
   <xacro:property name="mass"       value="0.061"/>
   <xacro:property name="collision_length_x"   value="${2.25*cm2m}" />
@@ -10,27 +11,10 @@
   <xacro:property name="collision_offset_y"   value="${0*cm2m}" />
   <xacro:property name="collision_offset_z"   value="${-0.5*cm2m}" />
-  <joint name="${name}_joint" type="fixed">
-    <parent link="${parent_link}"/>
-    <child link="${name}_link"/>
-    <xacro:insert_block name="origin"/>
-  </joint>
-  <link name="${name}_link">
-    <visual>
-      <geometry>
-        <mesh filename="file://$(find turtlebot4_description)/meshes/OAK-D-Lite.STL" scale="0.001 0.001 0.001" />
-      </geometry>
-    </visual>
-    <collision>
-      <origin xyz="${collision_offset_x} ${collision_offset_y} ${collision_offset_z}"/>
-      <geometry>
-        <box size="${collision_length_x} ${collision_length_y} ${collision_length_z}"/>
-      </geometry>
-    </collision>
-    <inertial>
-      <mass value="${mass}"/>
-      <inertia ixx="0.00000202475" ixy="0.0" ixz="0.0"
-	             iyy="0.00001527320" iyz="0.0" izz="0.00001605536" />
-    </inertial>
-  </link>
+  <xacro:property name="camera_model"  value="OAK-D-LITE" />
+  <xacro:property name="base_frame"    value="${name}_link" />
+  <xacro:depthai_camera camera_name="${name}" parent="${parent_link}"
+                        camera_model="${camera_model}" base_frame="${base_frame}"
+                        cam_pos_x="${cam_pos_x}" cam_pos_y="${cam_pos_y}" cam_pos_z="${cam_pos_z}"
+                        cam_roll="${cam_roll}" cam_pitch="${cam_pitch}" cam_yaw="${cam_yaw}"/>
   <gazebo reference="${name}_link">
     <sensor name="rgbd_camera" type="rgbd_camera">

Commit message: Using depthai camera macro for oakd pro and lite Using package:// instead of file:// for finding mesh files

File: turtlebot4_description/urdf/lite/turtlebot4.urdf.xacro (robot description, xacro)
@@ -28,5 +28,4 @@
                    cam_pos_y="${oakd_lite_y_offset}"
                    cam_pos_z="${oakd_lite_z_offset}"
-                   cam_roll="0.0" cam_pitch="0.0" cam_yaw="0.0">
-  </xacro:oakd_lite>
+                   cam_roll="0.0" cam_pitch="0.0" cam_yaw="0.0"/>
 </robot>

File: turtlebot4_description/urdf/sensors/camera_bracket.urdf.xacro (robot description, xacro)
@@ -14,5 +14,5 @@
     <visual>
       <geometry>
-       <mesh filename="file://$(find turtlebot4_description)/meshes/camera_bracket.STL" scale="0.001 0.001 0.001" />
+       <mesh filename="package://turtlebot4_description/meshes/camera_bracket.STL" scale="0.001 0.001 0.001" />
       </geometry>
     </visual>

File: turtlebot4_description/urdf/sensors/oakd_pro.urdf.xacro (robot description, xacro)
@@ -1,6 +1,7 @@
 <?xml version="1.0"?>
 <robot xmlns:xacro="http://ros.org/wiki/xacro">
-<xacro:macro name="oakd_pro" params="name parent_link *origin">
+<xacro:macro name="oakd_pro" params="name parent_link cam_pos_x cam_pos_y cam_pos_z cam_roll cam_pitch cam_yaw">
   <xacro:include filename="$(find irobot_create_description)/urdf/common_properties.urdf.xacro"/>
+  <xacro:include filename="$(find depthai_bridge)/urdf/include/depthai_macro.urdf.xacro"/>
   <xacro:property name="mass"       value="0.061"/>
   <xacro:property name="collision_length_x"   value="${2.25*cm2m}" />
@@ -10,27 +11,10 @@
   <xacro:property name="collision_offset_y"   value="${0*cm2m}" />
   <xacro:property name="collision_offset_z"   value="${-0.5*cm2m}" />
-  <joint name="${name}_joint" type="fixed">
-    <parent link="${parent_link}"/>
-    <child link="${name}_link"/>
-    <xacro:insert_block name="origin"/>
-  </joint>
-  <link name="${name}_link">
-    <visual>
-      <geometry>
-        <mesh filename="file://$(find turtlebot4_description)/meshes/OAK-D-Pro.STL" scale="0.001 0.001 0.001" />
-      </geometry>
-    </visual>
-    <collision>
-      <origin xyz="${collision_offset_x} ${collision_offset_y} ${collision_offset_z}"/>
-      <geometry>
-        <box size="${collision_length_x} ${collision_length_y} ${collision_length_z}"/>
-      </geometry>
-    </collision>
-    <inertial>
-      <mass value="${mass}"/>
-      <inertia ixx="0.00000202475" ixy="0.0" ixz="0.0"
-	             iyy="0.00001527320" iyz="0.0" izz="0.00001605536" />
-    </inertial>
-  </link>
+  <xacro:property name="camera_model"  value="OAK-D-PRO" />
+  <xacro:property name="base_frame"    value="${name}_link" />
+  <xacro:depthai_camera camera_name="${name}" parent="${parent_link}"
+                        camera_model="${camera_model}" base_frame="${base_frame}"
+                        cam_pos_x="${cam_pos_x}" cam_pos_y="${cam_pos_y}" cam_pos_z="${cam_pos_z}"
+                        cam_roll="${cam_roll}" cam_pitch="${cam_pitch}" cam_yaw="${cam_yaw}"/>
   <gazebo reference="${name}_link">
     <sensor name="rgbd_camera" type="rgbd_camera">

File: turtlebot4_description/urdf/sensors/rplidar.urdf.xacro (robot description, xacro)
@@ -18,5 +18,5 @@
     <visual>
       <geometry>
-        <mesh filename="file://$(find turtlebot4_description)/meshes/rplidar.STL" scale="0.001 0.001 0.001" />
+        <mesh filename="package://turtlebot4_description/meshes/rplidar.STL" scale="0.001 0.001 0.001" />
       </geometry>
     </visual>

File: turtlebot4_description/urdf/standard/tower_sensor_plate.urdf.xacro (robot description, xacro)
@@ -14,5 +14,5 @@
     <visual>
       <geometry>
-       <mesh filename="file://$(find turtlebot4_description)/meshes/tower_sensor_plate.STL" scale="0.001 0.001 0.001" />
+       <mesh filename="package://turtlebot4_description/meshes/tower_sensor_plate.STL" scale="0.001 0.001 0.001" />
       </geometry>
     </visual>

File: turtlebot4_description/urdf/standard/tower_standoff.urdf.xacro (robot description, xacro)
@@ -15,5 +15,5 @@
       <origin rpy="0 ${pi/2} 0"/>
       <geometry>
-       <mesh filename="file://$(find turtlebot4_description)/meshes/tower_standoff.STL" scale="0.001 0.001 0.001" />
+       <mesh filename="package://turtlebot4_description/meshes/tower_standoff.STL" scale="0.001 0.001 0.001" />
       </geometry>
     </visual>

File: turtlebot4_description/urdf/standard/turtlebot4.urdf.xacro (robot description, xacro)
@@ -43,10 +43,10 @@
       <origin xyz="0 0 0" rpy="${pi/2} 0 ${pi/2}"/>
       <geometry>
-        <mesh filename="file://$(find turtlebot4_description)/meshes/shell.STL" scale="0.001 0.001 0.001" />
+        <mesh filename="package://turtlebot4_description/meshes/shell.STL" scale="0.001 0.001 0.001" />
       </geometry>
     </visual>
     <collision name="shell_collision">
       <geometry>
-        <mesh filename="file://$(find turtlebot4_description)/meshes/shell_collision.STL" scale="0.001 0.001 0.001" />
+        <mesh filename="package://turtlebot4_description/meshes/shell_collision.STL" scale="0.001 0.001 0.001" />
       </geometry>
     </collision>
@@ -98,6 +98,8 @@
     <origin xyz="${camera_mount_x_offset} ${camera_mount_y_offset} ${camera_mount_z_offset}"/>
   </xacro:camera_bracket>
-  <xacro:oakd_pro name="oakd_pro" parent_link="oakd_pro_camera_bracket">
-    <origin xyz="${oakd_pro_x_offset} ${oakd_pro_y_offset} ${oakd_pro_z_offset}"/>
-  </xacro:oakd_pro>
+  <xacro:oakd_pro name="oakd_pro" parent_link="oakd_pro_camera_bracket"
+                  cam_pos_x="${oakd_pro_x_offset}"
+                  cam_pos_y="${oakd_pro_y_offset}"
+                  cam_pos_z="${oakd_pro_z_offset}"
+                  cam_roll="0.0" cam_pitch="0.0" cam_yaw="0.0"/>
 </robot>

File: turtlebot4_description/urdf/standard/weight_block.urdf.xacro (robot description, xacro)
@@ -14,5 +14,5 @@
     <visual>
       <geometry>
-       <mesh filename="file://$(find turtlebot4_description)/meshes/weight_block.STL" scale="0.001 0.001 0.001" />
+       <mesh filename="package://turtlebot4_description/meshes/weight_block.STL" scale="0.001 0.001 0.001" />
       </geometry>
     </visual>

Commit message: Updated gazebo reference link

File: turtlebot4_description/urdf/lite/turtlebot4.urdf.xacro (robot description, xacro)
@@ -13,5 +13,5 @@
   <xacro:property name="camera_mount_y_offset"         value="${0*cm2m}"/>
   <xacro:property name="camera_mount_z_offset"         value="${2.914772*cm2m}"/>
-  <xacro:property name="oakd_lite_x_offset"             value="${5.294026*cm2m}"/>
+  <xacro:property name="oakd_lite_x_offset"             value="${5.1*cm2m}"/>
   <xacro:property name="oakd_lite_y_offset"             value="${0*cm2m}"/>
   <xacro:property name="oakd_lite_z_offset"             value="${9.25385*cm2m}"/>

File: turtlebot4_description/urdf/sensors/oakd_lite.urdf.xacro (robot description, xacro)
@@ -17,5 +17,5 @@
                         cam_pos_x="${cam_pos_x}" cam_pos_y="${cam_pos_y}" cam_pos_z="${cam_pos_z}"
                         cam_roll="${cam_roll}" cam_pitch="${cam_pitch}" cam_yaw="${cam_yaw}"/>
-  <gazebo reference="${name}_link">
+  <gazebo reference="${name}_rgb_camera_optical_frame">
     <sensor name="rgbd_camera" type="rgbd_camera">
       <camera>

File: turtlebot4_description/urdf/sensors/oakd_pro.urdf.xacro (robot description, xacro)
@@ -17,5 +17,5 @@
                         cam_pos_x="${cam_pos_x}" cam_pos_y="${cam_pos_y}" cam_pos_z="${cam_pos_z}"
                         cam_roll="${cam_roll}" cam_pitch="${cam_pitch}" cam_yaw="${cam_yaw}"/>
-  <gazebo reference="${name}_link">
+  <gazebo reference="${name}_rgb_camera_optical_frame">
     <sensor name="rgbd_camera" type="rgbd_camera">
       <camera>
@@ -36,5 +36,5 @@
     <xacro:material_darkgray/>
   </gazebo>
-  <gazebo reference="${name}_joint">
+  <gazebo reference="${name}_center_joint">
     <preserveFixedJoint>true</preserveFixedJoint>
   </gazebo>

Commit message: Created oakd macro for both lite and pro. Added optical links. Switched to .dae meshes to fix Rviz issues

File: turtlebot4_description/urdf/lite/turtlebot4.urdf.xacro (robot description, xacro)
@@ -4,5 +4,5 @@
   <xacro:include filename="$(find irobot_create_description)/urdf/create3.urdf.xacro" />
   <xacro:include filename="$(find turtlebot4_description)/urdf/sensors/rplidar.urdf.xacro" />
-  <xacro:include filename="$(find turtlebot4_description)/urdf/sensors/oakd_lite.urdf.xacro" />
+  <xacro:include filename="$(find turtlebot4_description)/urdf/sensors/oakd.urdf.xacro" />
   <xacro:include filename="$(find turtlebot4_description)/urdf/sensors/camera_bracket.urdf.xacro" />
   <!-- Mechanical properties -->
@@ -13,5 +13,5 @@
   <xacro:property name="camera_mount_y_offset"         value="${0*cm2m}"/>
   <xacro:property name="camera_mount_z_offset"         value="${2.914772*cm2m}"/>
-  <xacro:property name="oakd_lite_x_offset"             value="${5.1*cm2m}"/>
+  <xacro:property name="oakd_lite_x_offset"             value="${5.294026*cm2m}"/>
   <xacro:property name="oakd_lite_y_offset"             value="${0*cm2m}"/>
   <xacro:property name="oakd_lite_z_offset"             value="${9.25385*cm2m}"/>
@@ -24,8 +24,6 @@
     <origin xyz="${camera_mount_x_offset} ${camera_mount_y_offset} ${camera_mount_z_offset + base_link_z_offset}"/>
   </xacro:camera_bracket>
-  <xacro:oakd_lite name="oakd_lite" parent_link="oakd_lite_camera_bracket"
-                   cam_pos_x="${oakd_lite_x_offset}"
-                   cam_pos_y="${oakd_lite_y_offset}"
-                   cam_pos_z="${oakd_lite_z_offset}"
-                   cam_roll="0.0" cam_pitch="0.0" cam_yaw="0.0"/>
+  <xacro:oakd name="oakd_lite" parent_link="oakd_lite_camera_bracket">
+    <origin xyz="${oakd_lite_x_offset} ${oakd_lite_y_offset} ${oakd_lite_z_offset}"/>
+  </xacro:oakd>
 </robot>

File: turtlebot4_description/urdf/sensors/camera_bracket.urdf.xacro (robot description, xacro)
@@ -14,5 +14,5 @@
     <visual>
       <geometry>
-       <mesh filename="package://turtlebot4_description/meshes/camera_bracket.STL" scale="0.001 0.001 0.001" />
+       <mesh filename="package://turtlebot4_description/meshes/camera_bracket.dae" scale="1 1 1" />
       </geometry>
     </visual>

File: turtlebot4_description/urdf/sensors/rplidar.urdf.xacro (robot description, xacro)
@@ -18,5 +18,5 @@
     <visual>
       <geometry>
-        <mesh filename="package://turtlebot4_description/meshes/rplidar.STL" scale="0.001 0.001 0.001" />
+        <mesh filename="package://turtlebot4_description/meshes/rplidar.dae" scale="1 1 1" />
       </geometry>
     </visual>

File: turtlebot4_description/urdf/standard/tower_sensor_plate.urdf.xacro (robot description, xacro)
@@ -14,5 +14,5 @@
     <visual>
       <geometry>
-       <mesh filename="package://turtlebot4_description/meshes/tower_sensor_plate.STL" scale="0.001 0.001 0.001" />
+       <mesh filename="package://turtlebot4_description/meshes/tower_sensor_plate.dae" scale="1 1 1" />
       </geometry>
     </visual>

File: turtlebot4_description/urdf/standard/tower_standoff.urdf.xacro (robot description, xacro)
@@ -15,5 +15,5 @@
       <origin rpy="0 ${pi/2} 0"/>
       <geometry>
-       <mesh filename="package://turtlebot4_description/meshes/tower_standoff.STL" scale="0.001 0.001 0.001" />
+       <mesh filename="package://turtlebot4_description/meshes/tower_standoff.dae" scale="1 1 1" />
       </geometry>
     </visual>

File: turtlebot4_description/urdf/standard/turtlebot4.urdf.xacro (robot description, xacro)
@@ -4,5 +4,5 @@
   <xacro:include filename="$(find irobot_create_description)/urdf/create3.urdf.xacro" />
   <xacro:include filename="$(find turtlebot4_description)/urdf/sensors/rplidar.urdf.xacro" />
-  <xacro:include filename="$(find turtlebot4_description)/urdf/sensors/oakd_pro.urdf.xacro" />
+  <xacro:include filename="$(find turtlebot4_description)/urdf/sensors/oakd.urdf.xacro" />
   <xacro:include filename="$(find turtlebot4_description)/urdf/sensors/camera_bracket.urdf.xacro" />
   <xacro:include filename="$(find turtlebot4_description)/urdf/standard/tower_standoff.urdf.xacro" />
@@ -43,10 +43,10 @@
       <origin xyz="0 0 0" rpy="${pi/2} 0 ${pi/2}"/>
       <geometry>
-        <mesh filename="package://turtlebot4_description/meshes/shell.STL" scale="0.001 0.001 0.001" />
+        <mesh filename="package://turtlebot4_description/meshes/shell.dae" scale="1 1 1" />
       </geometry>
     </visual>
     <collision name="shell_collision">
       <geometry>
-        <mesh filename="package://turtlebot4_description/meshes/shell_collision.STL" scale="0.001 0.001 0.001" />
+        <mesh filename="package://turtlebot4_description/meshes/shell_collision.dae" scale="1 1 1" />
       </geometry>
     </collision>
@@ -98,8 +98,6 @@
     <origin xyz="${camera_mount_x_offset} ${camera_mount_y_offset} ${camera_mount_z_offset}"/>
   </xacro:camera_bracket>
-  <xacro:oakd_pro name="oakd_pro" parent_link="oakd_pro_camera_bracket"
-                  cam_pos_x="${oakd_pro_x_offset}"
-                  cam_pos_y="${oakd_pro_y_offset}"
-                  cam_pos_z="${oakd_pro_z_offset}"
-                  cam_roll="0.0" cam_pitch="0.0" cam_yaw="0.0"/>
+  <xacro:oakd name="oakd_pro" parent_link="oakd_pro_camera_bracket">
+    <origin xyz="${oakd_pro_x_offset} ${oakd_pro_y_offset} ${oakd_pro_z_offset}"/>
+  </xacro:oakd>
 </robot>

File: turtlebot4_description/urdf/standard/weight_block.urdf.xacro (robot description, xacro)
@@ -14,5 +14,5 @@
     <visual>
       <geometry>
-       <mesh filename="package://turtlebot4_description/meshes/weight_block.STL" scale="0.001 0.001 0.001" />
+       <mesh filename="package://turtlebot4_description/meshes/weight_block.dae" scale="1 1 1" />
       </geometry>
     </visual>
